File: SHO-V1.1.sch (EAGLE design)
At the start: 16 parts, among them Q1 BS170

Commit message: New schematic and Board layout
Parts:
- +9V: device gm-supply:+9V(T) -> mb_supply:+9V(T)
- C1: device gm-caps-film-box:072X0352 -> mb_caps-chicklet:075X0302
- C2, C3: device gm-caps-electro-pol:0631 -> mb_caps-electro:0631
- D1: device gm-diodes:1N9ZENER -> mb_diodes:1N9ZENER
- GND: device gm-supply:GND(T) -> mb_supply:GND(T)
- IN: device gm-supply:IN(T) -> mb_supply:IN(T)
- LED: device gm-supply:PAD -> mb_supply:PAD
- OUT: device gm-supply:OUT(T) -> mb_supply:OUT(T)
- POT1: device gm-pots:POT16MM -> mb_pots:POT16MM_PCB_PADS
- Q1: device gm-trans:BS170 -> mb_trans:BS170
- R1, R2, R3, R4, R5: device gm-resistors:6MM.3 -> mb_resistors:6MM.3
Other:
- note added: "Xenocoder Right Side Boost V 1.1 11.2013"
Changed lines of the file:
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@@
 </classes>
 <parts>
-<part name="IN" library="gm-supply" deviceset="IN(T)" device=""/>
-<part name="OUT" library="gm-supply" deviceset="OUT(T)" device=""/>
-<part name="+9V" library="gm-supply" deviceset="+9V(T)" device=""/>
-<part name="GND" library="gm-supply" deviceset="GND(T)" device=""/>
+<part name="IN" library="mb_supply" deviceset="IN(T)" device=""/>
+<part name="OUT" library="mb_supply" deviceset="OUT(T)" device=""/>
+<part name="+9V" library="mb_supply" deviceset="+9V(T)" device=""/>
+<part name="GND" library="mb_supply" deviceset="GND(T)" device=""/>
 <part name="GND2" library="gm-supply" deviceset="GND" device=""/>
 <part name="GND3" library="gm-supply" deviceset="GND" device=""/>
-<part name="R1" library="gm-resistors" deviceset="6MM" device=".3" value="10M"/>
-<part name="R3" library="gm-resistors" deviceset="6MM" device=".3" value="5k1"/>
-<part name="R2" library="gm-resistors" deviceset="6MM" device=".3" value="10M"/>
-<part name="R4" library="gm-resistors" deviceset="6MM" device=".3" value="100k"/>
-<part name="C3" library="gm-caps-electro-pol" deviceset="063" device="1" value="10uF"/>
-<part name="C1" library="gm-caps-film-box" deviceset="072X035" device="2" value="100nF"/>
-<part name="D1" library="gm-diodes" deviceset="1N9*ZENER" device="" value="9.1Zener"/>
-<part name="POT1" library="gm-pots" deviceset="POT" device="16MM" value="C5k"/>
-<part name="Q1" library="gm-trans" deviceset="BS170" device=""/>
-<part name="C2" library="gm-caps-electro-pol" deviceset="063" device="1" value="47uF"/>
+<part name="R1" library="mb_resistors" deviceset="6MM" device=".3" value="10M"/>
+<part name="R3" library="mb_resistors" deviceset="6MM" device=".3" value="5k1"/>
+<part name="R2" library="mb_resistors" deviceset="6MM" device=".3" value="10M"/>
+<part name="R4" library="mb_resistors" deviceset="6MM" device=".3" value="100k"/>
+<part name="C3" library="mb_caps-electro" deviceset="063" device="1" value="10uF"/>
+<part name="C1" library="mb_caps-chicklet" deviceset="075X030" device="2" value="100nF"/>
+<part name="D1" library="mb_diodes" deviceset="1N9*ZENER" device="" value="9.1Zener"/>
+<part name="POT1" library="mb_pots" deviceset="POT" device="16MM_PCB_PADS" value="C5k"/>
+<part name="Q1" library="mb_trans" deviceset="BS170" device=""/>
+<part name="C2" library="mb_caps-electro" deviceset="063" device="1" value="47uF"/>
 <part name="GND4" library="gm-supply" deviceset="GND" device=""/>
-<part name="R5" library="gm-resistors" deviceset="6MM" device=".3" value="2k2"/>
-<part name="LED" library="gm-supply" deviceset="PAD" device="" value="3mm"/>
+<part name="R5" library="mb_resistors" deviceset="6MM" device=".3" value="2k2"/>
+<part name="LED" library="mb_supply" deviceset="PAD" device="" value="3mm"/>
 </parts>
 <sheets>
 <sheet>
 <plain>
+<text x="0" y="45.72" size="1.778" layer="91">Xenocoder
+Right Side Boost
+V 1.1 11.2013</text>
 </plain>
 <instances>
@@
 </schematic>
 </drawing>
+<compatibility>
+<note version="6.3" minversion="6.2.2" severity="warning">
+Since Version 6.2.2 text objects can contain more than one line,
+which will not be processed correctly with this version.
+</note>
+</compatibility>
 </eagle>
