File: SHO.sch (EAGLE design)
At the start: 16 parts, among them Q1 BS170

Commit message: Updated layout
Parts:
- added G: GND(T), mb_supply:GND(T)
- added L: 3mm, mb_supply:PAD
- LED: value 3mm -> LED3MM; device mb_supply:PAD -> mb_diodes:LED3MM
Connections:
- new net N$5: L.PAD, LED.C
- net GND: now also G.GND
- net N$4: now also LED.A; no longer LED.PAD
Changed lines of the file:
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@@
 <?xml version="1.0" encoding="utf-8"?>
 <!DOCTYPE eagle SYSTEM "eagle.dtd">
-<eagle version="6.4">
+<eagle version="7.1.0">
 <drawing>
 <settings>
@@
 <part name="+9V" library="mb_supply" deviceset="+9V(T)" device=""/>
 <part name="GND" library="mb_supply" deviceset="GND(T)" device=""/>
-<part name="GND2" library="gm-supply" deviceset="GND" device=""/>
 <part name="GND3" library="gm-supply" deviceset="GND" device=""/>
 <part name="R1" library="mb_resistors" deviceset="6MM" device=".3" value="10M"/>
@@
 <part name="GND4" library="gm-supply" deviceset="GND" device=""/>
 <part name="R5" library="mb_resistors" deviceset="6MM" device=".3" value="2k2"/>
-<part name="LED" library="mb_supply" deviceset="PAD" device="" value="3mm"/>
+<part name="L" library="mb_supply" deviceset="PAD" device="" value="3mm"/>
+<part name="LED" library="mb_diodes" deviceset="LED" device="3MM"/>
+<part name="G" library="mb_supply" deviceset="GND(T)" device=""/>
 </parts>
 <sheets>
@@
 <instance part="+9V" gate="+9V" x="40.64" y="96.52"/>
 <instance part="GND" gate="GND" x="27.94" y="27.94"/>
-<instance part="GND2" gate="GND" x="68.58" y="43.18"/>
 <instance part="GND3" gate="GND" x="40.64" y="27.94"/>
 <instance part="R1" gate="G$1" x="27.94" y="71.12" rot="R90"/>
@@
 <instance part="GND4" gate="GND" x="15.24" y="81.28"/>
 <instance part="R5" gate="G$1" x="53.34" y="88.9"/>
-<instance part="LED" gate="G$1" x="66.04" y="88.9"/>
+<instance part="L" gate="G$1" x="78.74" y="88.9"/>
+<instance part="LED" gate="G$1" x="68.58" y="88.9" rot="R180"/>
+<instance part="G" gate="GND" x="68.58" y="43.18"/>
 </instances>
 <busses>
@@
 </net>
 <net name="GND" class="0">
-<segment>
-<pinref part="GND2" gate="GND" pin="GND"/>
-<pinref part="R4" gate="G$1" pin="1"/>
-<wire x1="68.58" y1="45.72" x2="68.58" y2="53.34" width="0.1524" layer="91"/>
-</segment>
 <segment>
 <pinref part="POT1" gate="G$1" pin="1"/>
@@
 <wire x1="22.86" y1="88.9" x2="15.24" y2="88.9" width="0.1524" layer="91"/>
 <wire x1="15.24" y1="88.9" x2="15.24" y2="83.82" width="0.1524" layer="91"/>
+</segment>
+<segment>
+<pinref part="R4" gate="G$1" pin="1"/>
+<wire x1="68.58" y1="45.72" x2="68.58" y2="53.34" width="0.1524" layer="91"/>
+<pinref part="G" gate="GND" pin="GND"/>
 </segment>
 </net>
@@
 <segment>
 <pinref part="R5" gate="G$1" pin="2"/>
-<pinref part="LED" gate="G$1" pin="PAD"/>
+<pinref part="LED" gate="G$1" pin="A"/>
 <wire x1="58.42" y1="88.9" x2="63.5" y2="88.9" width="0.1524" layer="91"/>
 </segment>
 </net>
+<net name="N$5" class="0">
+<segment>
+<pinref part="LED" gate="G$1" pin="C"/>
+<pinref part="L" gate="G$1" pin="PAD"/>
+<wire x1="71.12" y1="88.9" x2="76.2" y2="88.9" width="0.1524" layer="91"/>
+</segment>
+</net>
